File: Cuspid40/Cuspid40.kicad_pcb (KiCad board)
At the start: 2 copper layers, 276.2 x 91 mm, 154 parts, among them U1 Pluto

Commit message: Updated some files
Parts:
- moved MX30 4.67 mm to (317.6, 129.8)
Routing:
- net row0: track 257.1 -> 275.4 mm
- net Net-(D27-A): track 15.5 -> 17.5 mm
- net col12: track 242.9 -> 241.3 mm
